File: pcb/pir_pcb/PIR Board/PIR Board/tinyScrubCam_pcb/tinyScrubCam_pcb/tinyScrubCam_pcb.kicad_sch (KiCad schematic)
At the start: 16 parts, among them U1 AP2112K-3.3, U2 LM393

Commit message: update
Parts:
- removed C1, C2: 10uF, symbol Device:C
- removed J_BAT1: Conn_01x02, symbol Connector_Generic:Conn_01x02
- removed U1: AP2112K-3.3, Package_TO_SOT_SMD:SOT-23-5, symbol Regulator_Linear:AP2112K-3.3
- added J_IR_FLASH1, J_IR_PWR1, J_PWR_IN1: Conn_01x02, Connector_PinHeader_2.54mm:PinHeader_1x02_P2.54mm_Vertical, symbol Connector_Generic:Conn_01x02
- added Q1: D44H8, Package_TO_SOT_THT:TO-220-3_Vertical, symbol Transistor_BJT:Q_NPN_BCE
- added RPD1: 100k, Resistor_THT:R_Axial_DIN0207_L6.3mm_D2.5mm_P10.16mm_Horizontal, symbol Device:R
- added R_BASE1: 200, Resistor_THT:R_Axial_DIN0207_L6.3mm_D2.5mm_P10.16mm_Horizontal, symbol Device:R
- J_ESP32_L1, J_ESP32_R1: footprint (none) -> Connector_PinHeader_2.54mm:PinHeader_1x20_P2.54mm_Vertical
- J_LORA_GPIO1: footprint (none) -> Connector_PinHeader_2.54mm:PinHeader_1x05_P2.54mm_Vertical
- J_LORA_MAIN1: footprint (none) -> Connector_PinHeader_2.54mm:PinHeader_1x09_P2.54mm_Vertical
- J_PIR1: footprint (none) -> Connector_PinHeader_2.54mm:PinHeader_1x03_P2.54mm_Vertical
- R1, R2, R3, R4, RHYS1, RPU1: footprint (none) -> Resistor_THT:R_Axial_DIN0207_L6.3mm_D2.5mm_P10.16mm_Horizontal
- U2: footprint (none) -> Package_DIP:DIP-8_W7.62mm
Connections:
- net 3V3: now also J_ESP32_L1.1 (3V3), J_LORA_MAIN1.1 (3V3), J_LORA_MAIN1.3 (EN); no longer J_LORA_MAIN1.EN, J_LORA_MAIN1.VIN (3V3)
- net GND: now also J_ESP32_R1.20 (GND), J_LORA_MAIN1.2 (GND), J_IR_PWR1.2 (Pin_2), J_PWR_IN1.2 (Pin_2), Q1.3 (E), RPD1.2; no longer J_ESP32_R1.GND, J_LORA_MAIN1.GND
- net LORA_CS: now also J_ESP32_L1.12 (GPIO3), J_LORA_MAIN1.8 (CS); no longer J_ESP32_L1.3 (GPIO3), J_LORA_MAIN1.CS
- net LORA_G0: now also J_ESP32_R1.18 (GPIO20), J_LORA_MAIN1.4 (GPIO0); no longer J_ESP32_R1.20 (GPIO20), J_LORA_MAIN1.G0 (GPIO0)
- net LORA_G1: now also J_ESP32_R1.17 (GPIO21), J_LORA_GPIO1.1 (GPIO1); no longer J_ESP32_R1.21 (GPIO21), J_LORA_GPIO1.G1 (GPIO1)
- net LORA_MISO: now also J_ESP32_R1.16 (GPIO47), J_LORA_MAIN1.6 (MISO); no longer J_ESP32_R1.47 (GPIO47), J_LORA_MAIN1.MISO
- net LORA_MOSI: now also J_LORA_MAIN1.7 (MOSI); no longer J_LORA_MAIN1.MOSI
- net LORA_RST: now also J_ESP32_L1.19 (GPIO14), J_LORA_MAIN1.9 (RST); no longer J_ESP32_L1.14 (GPIO14), J_LORA_MAIN1.RST
- net LORA_SCK: now also J_ESP32_R1.14 (GPIO45), J_LORA_MAIN1.5 (SCK); no longer J_ESP32_R1.45 (GPIO45), J_LORA_MAIN1.SCK
- net PIR_OUT: now also J_ESP32_R1.3 (GPIO1); no longer J_ESP32_R1.1 (GPIO1)
- new net IR_EN: J_ESP32_L1.3 (GPIO4), Q1.1 (B), RPD1.1, R_BASE1.1, R_BASE1.2
- new net IR_PWR: J_IR_FLASH1.1 (Pin_1), J_IR_PWR1.1 (Pin_1)
- new net IR_SW: J_IR_FLASH1.2 (Pin_2), Q1.2 (C)
- new net SYS_PWR: J_ESP32_L1.20 (5V), J_PWR_IN1.1 (Pin_1)
- no-connect marks 34 -> 32
Other:
- note added: "Power System (LiPo)"
- note removed: "Power System (LiPO -> 3.3V Regulation)"
- moved on the sheet: J_LORA_MAIN1
