File: pcb/tinyScrubCam_pcb/tinyScrubCam_pcb.kicad_pcb (KiCad board)
At the start: 2 copper layers, 117 x 76.2 mm, 22 parts, among them Q1 D44H8, U2 LM393

Commit message: update
Parts:
- added G***: LOGO, LOGO, F.Cu at (186.9, 128.7)
- J_PIR1: footprint Connector_PinHeader_2.54mm:PinHeader_1x03_P2.54mm_Vertical -> Connector_PinSocket_2.54mm:PinSocket_1x03_P2.54mm_Vertical
- J_PWR_IN1: footprint Connector_PinHeader_2.54mm:PinHeader_1x02_P2.54mm_Vertical -> Connector_JST:JST_PH_B2B-PH-K_1x02_P2.00mm_Vertical
- moved J_PIR1 19.8 mm to (205.5, 102.6), turned to 180 degrees
- moved J_PWR_IN1 1.86 mm to (159.7, 132.3), turned to 0 degrees
Routing:
- net /PIR_RAW: track 51.5 -> 24.5 mm
- net /3V3: track 133.3 -> 153.5 mm
- net /PIR_OUT: track 77.2 -> 70.9 mm
- net /SYS_PWR: track 14.9 -> 16.2 mm
Other:
- board text added: "ESP32-S3 WROOM"
- board text added: "LoRaWAN 915MHz"
- board text added: "Team"
- board text added: "Wildsight"
