File: pcb/tinyScrubCam_pcb  v1.1/tinyScrubCam_pcb  v1.1/tinyScrubCam_pcb.kicad_sch (KiCad schematic)
At the start: 18 parts, among them Q1 D44H8, U2 LM393

Commit message: pcb
Parts:
- added unit 2 of U2
- J_ESP32_L1, J_ESP32_R1: footprint (none) -> Connector_PinHeader_2.54mm:PinHeader_1x20_P2.54mm_Vertical
- J_IR_FLASH1, J_IR_PWR1: footprint (none) -> Connector_PinHeader_2.54mm:PinHeader_1x02_P2.54mm_Vertical
- J_LORA_GPIO1: footprint (none) -> Connector_PinHeader_2.54mm:PinHeader_1x05_P2.54mm_Vertical
- J_LORA_MAIN1: footprint (none) -> Connector_PinHeader_2.54mm:PinHeader_1x09_P2.54mm_Vertical
- J_PIR1: footprint (none) -> Connector_PinSocket_2.54mm:PinSocket_1x03_P2.54mm_Vertical
- J_PWR_IN1: footprint (none) -> Connector_JST:JST_PH_B2B-PH-K_1x02_P2.00mm_Vertical
- Q1: footprint (none) -> Package_TO_SOT_THT:TO-220-3_Vertical
- R1, R2, R4, RHYS1, RPD1, RPU1, R_BASE1: footprint (none) -> Resistor_THT:R_Axial_DIN0207_L6.3mm_D2.5mm_P10.16mm_Horizontal
- R3: footprint (none) -> Resistor_THT:R_Axial_DIN0207_L6.3mm_D2.5mm_P10.16mm_Horizontal; KiLib_Generator (none) -> resistor/THT
Connections:
- net 3V3: now also J_ESP32_L1.1 (3V3), J_LORA_MAIN1.1 (3V3), J_LORA_MAIN1.3 (EN); no longer J_LORA_MAIN1.EN, J_LORA_MAIN1.VIN (3V3)
- net GND: now also J_ESP32_R1.20 (GND), J_LORA_MAIN1.2 (GND), U2.5 (+), U2.6 (-); no longer J_ESP32_R1.GND, J_LORA_MAIN1.GND
- net IR_EN: now also J_ESP32_R1.4 (GPIO2), Q1.1 (B), RPD1.1, R_BASE1.2; no longer J_ESP32_L1.4 (GPIO4)
- net LORA_CS: now also J_ESP32_L1.12 (GPIO3), J_LORA_MAIN1.8 (CS); no longer J_ESP32_L1.3 (GPIO3), J_LORA_MAIN1.CS
- net LORA_G0: now also J_ESP32_R1.18 (GPIO20), J_LORA_MAIN1.4 (GPIO0); no longer J_ESP32_R1.20 (GPIO20), J_LORA_MAIN1.G0 (GPIO0)
- net LORA_G1: now also J_ESP32_R1.17 (GPIO21), J_LORA_GPIO1.1 (GPIO1); no longer J_ESP32_R1.21 (GPIO21), J_LORA_GPIO1.G1 (GPIO1)
- net LORA_MISO: now also J_ESP32_R1.16 (GPIO47), J_LORA_MAIN1.6 (MISO); no longer J_ESP32_R1.47 (GPIO47), J_LORA_MAIN1.MISO
- net LORA_MOSI: now also J_LORA_MAIN1.7 (MOSI); no longer J_LORA_MAIN1.MOSI
- net LORA_RST: now also J_ESP32_L1.19 (GPIO14), J_LORA_MAIN1.9 (RST); no longer J_ESP32_L1.14 (GPIO14), J_LORA_MAIN1.RST
- net LORA_SCK: now also J_ESP32_R1.14 (GPIO45), J_LORA_MAIN1.5 (SCK); no longer J_ESP32_R1.45 (GPIO45), J_LORA_MAIN1.SCK
- net PIR_OUT: now also J_ESP32_R1.3 (GPIO1); no longer J_ESP32_R1.1 (GPIO1)
- net SYS_PWR: now also J_ESP32_L1.20 (5V); no longer J_ESP32_L1.5V
- net at R3.2, R4.1: now also U2.2 (-); no longer U2.3 (+)
- net at R1.2, R2.1, RHYS1.1: now also U2.3 (+); no longer U2.2 (-)
- no-connect marks 32 -> 33
Other:
- moved on the sheet: J_LORA_MAIN1, R3, R4
