File: pcb/tinyScrubCam_pcb  v1.1/tinyScrubCam_pir/tinyScrubCam_pir/tinyScrubCam_pir.kicad_sch (KiCad schematic)
At the start: 2 parts, among them J1 Conn_01x03, U1 EKMC1603111

Commit message: pcb
Connections:
- net GND: now also J1.3 (Pin_3), U1.3 (GND); no longer J1.2 (Pin_2), U1.2 (GND)
- net PIR_RAW: now also J1.2 (Pin_2), U1.2 (ANALOG); no longer J1.3 (Pin_3), U1.3 (ANALOG)
